Commit message: Migrate control stack to rebuilt v2 arm; add robot_state_publisher/RViz
Core v2 migration: model-config package (facadebot_description) with a
fail-closed loader selecting the active arm (v1/v2), geometry baked
offline from the URDF into YAML so no node parses XML at runtime, and
kinematics.py rewritten for v2's out-of-plane joint_4 axis. All three
hand-measured numbers (joint centers, joint limits, tool-tip offset) are
now filled in and confirmed on the rebuilt hardware (limits_source:
measured).

Adds joint_state_publisher_node (/joint_states) and a new display.launch.py
(robot_state_publisher + rviz2) so the arm can be visualized in RViz,
alongside the existing bringup.launch.py for the control stack itself.
Also includes the earlier servo-bus diagnostic script
(scripts/check_servo_bus.py), the min-jerk/streaming firmware changes,
and updated tests.

Co-Authored-By: Claude Sonnet 5 <noreply@anthropic.com>

File: ros2_ws/src/facadebot_description/urdf/URDF_V2.urdf (robot description, URDF)
Before this commit: robot URDF_Test, 5 links, 4 joints
Links:
- link base_link: mass 0.185876111089366 -> 0.20537; geometry collision mesh filename=package://facadebot_description/meshes/v2/base_link.STL; visual mesh filename=package://facadebot_description/meshes/v2/base_link.STL
- link link_1: mass 0.0864426238517261 -> 0.10742; geometry collision mesh filename=package://facadebot_description/meshes/v2/link_1.STL; visual mesh filename=package://facadebot_description/meshes/v2/link_1.STL
- link link_2: mass 0.114185703128181 -> 0.12744; geometry collision mesh filename=package://facadebot_description/meshes/v2/link_2.STL; visual mesh filename=package://facadebot_description/meshes/v2/link_2.STL
- link link_3: mass 0.156185703128181 -> 0.13481; geometry collision mesh filename=package://facadebot_description/meshes/v2/link_3.STL; visual mesh filename=package://facadebot_description/meshes/v2/link_3.STL
- link link_4: mass 0.0427573671532661 -> 0.034066; geometry collision mesh filename=package://facadebot_description/meshes/v2/link_4.STL; visual mesh filename=package://facadebot_description/meshes/v2/link_4.STL
Joints:
- joint joint_1: axis 0 0 1 -> 0 0 -1; limit lower=0.0 upper=4.18878 effort=0 velocity=0 -> (none); origin xyz=0 0 0.10061 rpy=0 0 0 -> xyz=0.00039 0.00089 0.0403 rpy=0 0 0; type revolute -> continuous
- joint joint_2: limit lower=0.0 upper=4.18878 effort=0 velocity=0 -> (none); origin xyz=0 0 0 rpy=1.5708 -1.5708 0 -> xyz=0 -0.00014 0.06111 rpy=0 -1.5708 0; type revolute -> continuous
- joint joint_3: limit lower=0.0 upper=4.18878 effort=0 velocity=0 -> (none); origin xyz=0.12511 0 0 rpy=0 0 0 -> xyz=0.13511 -0.00014 0 rpy=0 0 0; type revolute -> continuous
- joint joint_4: limit lower=0.22 upper=4.0 effort=0 velocity=0 -> (none); origin xyz=0.16511 0 0 rpy=0 0 0 -> xyz=0.14011 0 -0.00076 rpy=-1.5708 0 0; type revolute -> continuous
